File: Electronics/eConBadge.kicad_pcb (KiCad board)
At the start: 2 copper layers, 77.1 x 84.7 mm, 18 parts

Commit message: New PCB
Parts:
- removed L_D_DIODE: DIOAD1036W78L470D235, eConBadge:DIOAD1036W78L470D235
- added 330 LED_DATA_R: R_Axial_DIN0204_L3.6mm_D1.6mm_P7.62mm_Horizontal, Resistor_THT:R_Axial_DIN0204_L3.6mm_D1.6mm_P7.62mm_Horizontal, B.Cu at (183.3, 57.5)
- added 74AHCT125 : 74AHCT125, 74AHCT125:DIP794W45P254L1930H508Q14, B.Cu at (155.5, 52.5)
Connections:
- ESP32 pad 10: SD_CS -> SD_MISO
- ESP32 pad 11: SD_MOSI -> SD_CLK
- ESP32 pad 12: SD_CLK -> SD_MOSI
- ESP32 pad 15: SD_MISO -> SD_CS
- ESP32 pad 8: LED_DATA -> LED_DATA_3V
- LEDConnector pad 2: LED_DATA -> LED_DATA_5V_OUT
- R1 220K pad 1: BATT_IN_GND -> BATT_IN_REG
- SDCardReader pad 1: GND -> VCC3.3
- SDCardReader pad 2: SD_MISO -> SD_CS
- SDCardReader pad 3: SD_CLK -> SD_MOSI
- SDCardReader pad 4: SD_MOSI -> SD_CLK
- SDCardReader pad 5: SD_CS -> SD_MISO
- SDCardReader pad 6: VCC3.3 -> GND
- UpBtn pad 2: VCC3.3 -> GND
Routing:
- net LED_DATA: track 33.6 -> 0.00 mm
- net VCC_5V: track 93.2 -> 125.2 mm
- net LED_DATA_5V_SHIFT: track 0.00 -> 23.9 mm
- net BATT_IN_REG: track 6.12 -> 26.5 mm
- net LED_DATA_3V: track 0.00 -> 11.4 mm
- net BATT_IN_GND: track 19.6 -> 11.9 mm
- net LED_DATA_5V_OUT: track 0.00 -> 5.53 mm
- net SD_MISO: track 8.46 -> 13.5 mm
- net SD_CS: track 13.5 -> 8.81 mm
- net BATT_IN_VCC: track 11.3 -> 12.1 mm
- net OLED_CLK: track 7.16 -> 7.88 mm
